Commit message: function full

File: src/open_manipulator/open_manipulator_x_description/ros2_control/open_manipulator_x_system.ros2_control.xacro (robot description, xacro)
@@ -1,6 +1,5 @@
 <?xml version="1.0"?>
 <robot xmlns:xacro="http://www.ros.org/wiki/xacro">
-  <xacro:macro name="open_manipulator_x_system" params="prefix arm_port_name:='/dev/ttyarm'
-  hand_port_name:='/dev/ttyhand' use_sim:=^|false use_fake_hardware:=^|false
+  <xacro:macro name="open_manipulator_x_system" params="prefix hand_port_name:='/dev/ttyhand' use_sim:=^|false use_fake_hardware:=^|false
   fake_sensor_commands:=^|false">
     <ros2_control name="hand" type="system">
@@ -399,206 +398,4 @@
       </gpio>
     </ros2_control>
-  <!-- 这里开始是机械臂的定义 -->
-  <ros2_control name="arm" type="system">
-      <xacro:if value="$(arg use_sim)">
-        <hardware>
-          <plugin>gazebo_ros2_control/GazeboSystem</plugin>
-        </hardware>
-      </xacro:if>
-      <xacro:unless value="$(arg use_sim)">
-        <hardware>
-          <xacro:if value="${use_fake_hardware}">
-            <plugin>fake_components/GenericSystem</plugin>
-            <param name="fake_sensor_commands">${fake_sensor_commands}</param>
-            <param name="state_following_offset">0.0</param>
-          </xacro:if>
-          <xacro:unless value="${use_fake_hardware}">
-            <plugin>dynamixel_hardware_interface/DynamixelHardware</plugin>
-            <!-- 这里定义端口名称 -->
-            <param name="port_name">${arm_port_name}</param>
-            <!-- 这里定义波特率 -->
-            <param name="baud_rate">1000000</param>
-            <param name="error_timeout_sec">0.2</param>
-            <param name="dynamixel_model_folder">/param/dxl_model</param>
-            <!-- 这里定义关节数量 -->
-            <param name="number_of_joints">7</param>
-            <param name="number_of_transmissions">7</param>
-            <!-- 关节矩阵的形状要与上面保持一致 -->
-            <param name="transmission_to_joint_matrix">
-              1,0,0,0,0,0,0,
-              0,1,0,0,0,0,0,
-              0,0,1,0,0,0,0,
-              0,0,0,1,0,0,0,
-              0,0,0,0,1,0,0,
-              0,0,0,0,0,1,0,
-              0,0,0,0,0,0,1
-            </param>
-             <!-- 关节矩阵 (20*20) -->
-            <param name="joint_to_transmission_matrix">
-              1,0,0,0,0,0,0,
-              0,1,0,0,0,0,0,
-              0,0,1,0,0,0,0,
-              0,0,0,1,0,0,0,
-              0,0,0,0,1,0,0,
-              0,0,0,0,0,1,0,
-              0,0,0,0,0,0,1
-            </param>
-            <!-- 这里定义电机更新频率 -->
-            <param name="ros_update_freq">50</param>
-            <param name="dynamixel_state_pub_msg_name">dynamixel_hardware_interface/dxl_state</param>
-            <param name="get_dynamixel_data_srv_name">dynamixel_hardware_interface/get_dxl_data</param>
-            <param name="set_dynamixel_data_srv_name">dynamixel_hardware_interface/set_dxl_data</param>
-            <param name="reboot_dxl_srv_name">dynamixel_hardware_interface/reboot_dxl</param>
-            <param name="set_dxl_torque_srv_name">dynamixel_hardware_interface/set_dxl_torque</param>
-          </xacro:unless>
-        </hardware>
-      </xacro:unless>
-      <joint name="${prefix}joint1">
-        <command_interface name="position"/>
-        <state_interface name="position"/>
-        <state_interface name="velocity"/>
-        <state_interface name="effort"/>
-      </joint>
-      <joint name="${prefix}joint2">
-        <command_interface name="position"/>
-        <state_interface name="position"/>
-        <state_interface name="velocity"/>
-        <state_interface name="effort"/>
-      </joint>
-      <joint name="${prefix}joint3">
-        <command_interface name="position"/>
-        <state_interface name="position"/>
-        <state_interface name="velocity"/>
-        <state_interface name="effort"/>
-      </joint>
-      <joint name="${prefix}joint4">
-        <command_interface name="position"/>
-        <state_interface name="position"/>
-        <state_interface name="velocity"/>
-        <state_interface name="effort"/>
-      </joint>
-      <joint name="${prefix}joint5">
-        <command_interface name="position"/>
-        <state_interface name="position"/>
-        <state_interface name="velocity"/>
-        <state_interface name="effort"/>
-      </joint>
-      <joint name="${prefix}joint6">
-        <command_interface name="position"/>
-        <state_interface name="position"/>
-        <state_interface name="velocity"/>
-        <state_interface name="effort"/>
-      </joint>
-      <joint name="${prefix}joint7">
-        <command_interface name="position"/>
-        <state_interface name="position"/>
-        <state_interface name="velocity"/>
-        <state_interface name="effort"/>
-      </joint>
-  <gpio name="dxl16">
-       <param name="type">dxl</param>
-       <param name="ID">16</param>
-       <command_interface name="Goal Position"/>
-       <state_interface name="Present Position"/>
-       <state_interface name="Present Velocity"/>
-       <state_interface name="Present Current"/>
-       <state_interface name="Torque Enable"/>
-       <state_interface name="Present Input Voltage"/>
-       <param name="Position P Gain">800</param>
-       <param name="Position I Gain">0</param>
-       <param name="Position D Gain">100</param>
-       <param name="Drive Mode">0</param>
-       <param name="Profile Velocity">45</param>
-      </gpio>
-      <gpio name="dxl17">
-       <param name="type">dxl</param>
-       <param name="ID">17</param>
-       <command_interface name="Goal Position"/>
-       <state_interface name="Present Position"/>
-       <state_interface name="Present Velocity"/>
-       <state_interface name="Present Current"/>
-       <state_interface name="Torque Enable"/>
-       <state_interface name="Present Input Voltage"/>
-       <param name="Position P Gain">700</param>
-       <param name="Position I Gain">0</param>
-       <param name="Position D Gain">100</param>
-       <param name="Drive Mode">0</param>
-       <param name="Profile Velocity">45</param>
-      </gpio>
-      <gpio name="dxl18">
-       <param name="type">dxl</param>
-       <param name="ID">18</param>
-       <command_interface name="Goal Position"/>
-       <state_interface name="Present Position"/>
-       <state_interface name="Present Velocity"/>
-       <state_interface name="Present Current"/>
-       <state_interface name="Torque Enable"/>
-       <state_interface name="Present Input Voltage"/>
-       <param name="Position P Gain">700</param>
-       <param name="Position I Gain">0</param>
-       <param name="Position D Gain">100</param>
-       <param name="Drive Mode">0</param>
-       <param name="Profile Velocity">45</param>
-      </gpio>
-      <gpio name="dxl19">
-       <param name="type">dxl</param>
-       <param name="ID">19</param>
-       <command_interface name="Goal Position"/>
-       <state_interface name="Present Position"/>
-       <state_interface name="Present Velocity"/>
-       <state_interface name="Present Current"/>
-       <state_interface name="Torque Enable"/>
-       <state_interface name="Present Input Voltage"/>
-       <param name="Position P Gain">700</param>
-       <param name="Position I Gain">0</param>
-       <param name="Position D Gain">0</param>
-       <param name="Drive Mode">0</param>
-       <param name="Profile Velocity">45</param>
-      </gpio>
-      <gpio name="dxl20">
-       <param name="type">dxl</param>
-       <param name="ID">20</param>
-       <command_interface name="Goal Position"/>
-       <state_interface name="Present Position"/>
-       <state_interface name="Present Velocity"/>
-       <state_interface name="Present Current"/>
-       <state_interface name="Torque Enable"/>
-       <state_interface name="Present Input Voltage"/>
-       <param name="Position P Gain">700</param>
-       <param name="Position I Gain">0</param>
-       <param name="Position D Gain">000</param>
-       <param name="Drive Mode">0</param>
-       <param name="Profile Velocity">45</param>
-      </gpio>
-      <gpio name="dxl21">
-       <param name="type">dxl</param>
-       <param name="ID">21</param>
-       <command_interface name="Goal Position"/>
-       <state_interface name="Present Position"/>
-       <state_interface name="Present Velocity"/>
-       <state_interface name="Present Current"/>
-       <state_interface name="Torque Enable"/>
-       <state_interface name="Present Input Voltage"/>
-       <param name="Position P Gain">600</param>
-       <param name="Position I Gain">0</param>
-       <param name="Position D Gain">0</param>
-       <param name="Drive Mode">0</param>
-       <param name="Profile Velocity">45</param>
-      </gpio>
-      <gpio name="dxl22">
-       <param name="type">dxl</param>
-       <param name="ID">22</param>
-       <command_interface name="Goal Position"/>
-       <state_interface name="Present Position"/>
-       <state_interface name="Present Velocity"/>
-       <state_interface name="Present Current"/>
-       <state_interface name="Torque Enable"/>
-       <state_interface name="Present Input Voltage"/>
-       <param name="Position P Gain">900</param>
-       <param name="Position I Gain">0</param>
-       <param name="Position D Gain">100</param>
-       <param name="Drive Mode">0</param>
-      </gpio>
-</ros2_control>
   </xacro:macro>
 </robot>

File: src/open_manipulator/open_manipulator_x_description/urdf/open_manipulator_x_robot.urdf.xacro (robot description, xacro)
@@ -7,5 +7,4 @@
   <xacro:arg name="fake_sensor_commands" default="false" />
   <!-- 端口定义 -->
-  <xacro:arg name="arm_port_name" default="/dev/ttyarm" />
   <xacro:arg name="hand_port_name" default="/dev/ttyhand" />
   <!-- Import Rviz colors -->
@@ -22,5 +21,4 @@
     use_fake_hardware="$(arg use_fake_hardware)"
     fake_sensor_commands="$(arg fake_sensor_commands)"
-    arm_port_name="$(arg arm_port_name)"
     hand_port_name="$(arg hand_port_name)"/>
   <!-- World -->
